File: PT4115-Miniboard.kicad_pcb (KiCad board)
At the start: 2 copper layers, 27 x 16.2 mm, 15 parts, among them J2 TestPoint, J3 TestPoint, J4 TestPoint, J5 TestPoint, J6 TestPoint, U1 PT4115

Commit message: update
Parts:
- moved C1 0.54 mm to (138.8, 106.5)
Routing:
- net /dim: track 16.1 -> 17.1 mm
Other:
- board text added: "DIM"
- board text added: "V-"
Changed lines of the file:
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@@
 	(footprint "Capacitor_SMD:C_0805_2012Metric"
 		(layer "F.Cu")
-		(at 138.25 106.7 90)
+		(at 138.75 106.5 90)
 		(descr "Capacitor SMD 0805 (2012 Metric), square (rectangular) end terminal, IPC_7351 nominal, (Body size source: IPC-SM-782 page 76, https://www.pcb-3d.com/wordpress/wp-content/uploads/ipc-sm-782a_amendment_1_and_2.pdf, https://docs.google.com/spreadsheets/d/1BsfQQcO9C6DZCsRaXUlFlo91Tg2WpOkGARC1WS5S8t0/edit?usp=sharing), generated with kicad-footprint-generator")
 		(tags "capacitor")
@@
 		)
 	)
+	(gr_text "DIM"
+		(at 132 110.5 0)
+		(layer "F.SilkS")
+		(effects
+			(font
+				(size 1 1)
+				(thickness 0.2)
+				(bold yes)
+			)
+			(justify left bottom)
+		)
+	)
 	(gr_text "L+\n"
 		(at 155.25 112.5 0)
@@
 	)
 	(gr_text "V+"
-		(at 137.95 102.7 0)
+		(at 136.75 102 0)
 		(layer "F.SilkS")
 		(effects
@@
 		)
 	)
+	(gr_text "V-"
+		(at 137.75 106.75 90)
+		(layer "F.SilkS")
+		(effects
+			(font
+				(size 1 1)
+				(thickness 0.2)
+				(bold yes)
+			)
+			(justify left bottom)
+		)
+	)
 	(segment
 		(start 150.0875 112)
@@
 	)
 	(segment
+		(start 138.1375 111.4)
+		(end 137.75 111.0125)
+		(width 0.3)
+		(layer "F.Cu")
+		(net 3)
+	)
+	(segment
+		(start 142.65 114.75)
+		(end 138.8 114.75)
+		(width 0.3)
+		(layer "F.Cu")
+		(net 3)
+	)
+	(segment
+		(start 138.8 114.75)
+		(end 137.15 113.1)
+		(width 0.3)
+		(layer "F.Cu")
+		(net 3)
+	)
+	(segment
+		(start 137.15 113.1)
+		(end 137.15 110.9)
+		(width 0.3)
+		(layer "F.Cu")
+		(net 3)
+	)
+	(segment
 		(start 135.8 107.45)
 		(end 135.75 107.5)
@@
 	)
 	(segment
-		(start 138.1375 111.4)
-		(end 137.75 111.0125)
-		(width 0.3)
-		(layer "F.Cu")
-		(net 3)
-	)
-	(segment
-		(start 142.65 114.75)
-		(end 138.8 114.75)
-		(width 0.3)
-		(layer "F.Cu")
-		(net 3)
-	)
-	(segment
-		(start 138.8 114.75)
-		(end 137.15 113.1)
-		(width 0.3)
-		(layer "F.Cu")
-		(net 3)
-	)
-	(segment
-		(start 137.15 113.1)
-		(end 137.15 110.9)
-		(width 0.3)
-		(layer "F.Cu")
-		(net 3)
-	)
-	(segment
 		(start 137.75 110.8125)
 		(end 137.0625 110.8125)
@@
 	)
 	(segment
-		(start 137.75 107.45)
+		(start 138.75 107.45)
 		(end 135.8 107.45)
 		(width 0.3)
